File: kicad/rgb_led_demo.kicad_sch (KiCad schematic)
At the start: 8 parts

Commit message: finish up creating schematics
Parts:
- added BT1: 4.5V, Battery:BatteryHolder_Keystone_2479_3xAAA, symbol Device:Battery_Cell
- added RVB1, RVG1: 10k Ohm, Potentiometer_THT:Potentiometer_Alps_RK163_Single_Horizontal, symbol Device:R_Potentiometer_Trim
- D1: renamed from D?; footprint (none) -> LED_THT:LED_D5.0mm-4_RGB
- RB1: renamed from R?; value R -> 68 Ohm; footprint (none) -> Resistor_THT:R_Axial_DIN0207_L6.3mm_D2.5mm_P7.62mm_Horizontal
- RG1: renamed from R?; value R -> 100 Ohm; footprint (none) -> Resistor_THT:R_Axial_DIN0207_L6.3mm_D2.5mm_P7.62mm_Horizontal
- RR1: renamed from R?; value R -> 120 Ohm; footprint (none) -> Resistor_THT:R_Axial_DIN0207_L6.3mm_D2.5mm_P7.62mm_Horizontal
- RVR1: renamed from RV?; value R_Potentiometer_Trim -> 10k Ohm; footprint (none) -> Potentiometer_THT:Potentiometer_Alps_RK163_Single_Horizontal
- SWB1, SWG1, SWR1: renamed from SW?; footprint (none) -> Button_Switch_THT:SW_DIP_SPSTx01_Slide_9.78x4.72mm_W7.62mm_P2.54mm
Connections:
- net GND: now also BT1.2 (-)
- net at RB1.2: now also RVB1.2
- net at RR1.2: now also RVR1.2; no longer RVR1.1
- net at RG1.2: now also RVG1.2
- net at D1.1 (RA): now also RVR1.3
- net at D1.2 (GA): now also RVG1.3
- net at D1.3 (BA): now also RVB1.3
- net +4V: no longer names the net of SWB1.1 (A), SWG1.1 (A), SWR1.1 (A)
- net +4V: now also BT1.1 (+)
Other:
- moved on the sheet: RB1, RR1, RVR1, SWB1, SWR1
